File: board/gb_1_0_pico.kicad_pcb (KiCad board)
At the start: 2 copper layers, 152.4 x 69.8 mm, 94 parts, among them J1 BMC, J2 EXPANSION, J3 2.8'' TFT LCD, J4 JACK_TRS, J5 MOTOR, J6 SPEAKER, Q1 IRLML6402, Q2 IRLML2502, Q3 IRLML6402, Q4 IRLML2502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

Commit message: dev@221123
Other:
- net class Default removed
- net class LogicPower removed
- net class Power removed
